File: step_down_led_board.sch (KiCad schematic (older format))
At the start: 34 parts, among them CON1 BARREL_JACK, J1 OSHW Logo, J2 Polarity Mark, M1 BuckModule, M2 BuckModule, P1 CONN_02X20, P2 CONN_01X02, P3 CONN_01X05, P4 CONN_01X02, P5 CONN_01X02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

Commit message: Use my solder jumper part.
Also fix some trace stragglers and silkscreen.
Parts:
- JP1, JP2, JP3, JP4, JP5, JP6, JP7, JP8: footprint jumper:SOLDER-JUMPER_1-WAY -> SolderJumpers-Tim:SJ_1_NO
Changed lines of the file:
@@
 LIBS:contrib
 LIBS:valves
-LIBS:buckmodule
 LIBS:step_down_led_board-cache
 EELAYER 25 0
@@
 F 0 "JP4" H 1850 6330 50  0000 C CNN
 F 1 "Jumper_NO_Small" H 1860 6190 50  0000 C CNN
-F 2 "jumper:SOLDER-JUMPER_1-WAY" H 1850 6250 50  0001 C CNN
+F 2 "SolderJumpers-Tim:SJ_1_NO" H 1850 6250 50  0001 C CNN
 F 3 "" H 1850 6250 50  0000 C CNN
 	1    1850 6250
@@
 F 0 "JP5" H 1850 6430 50  0000 C CNN
 F 1 "Jumper_NO_Small" H 1860 6290 50  0000 C CNN
-F 2 "jumper:SOLDER-JUMPER_1-WAY" H 1850 6350 50  0001 C CNN
+F 2 "SolderJumpers-Tim:SJ_1_NO" H 1850 6350 50  0001 C CNN
 F 3 "" H 1850 6350 50  0000 C CNN
 	1    1850 6350
@@
 F 0 "JP6" H 1850 6530 50  0000 C CNN
 F 1 "Jumper_NO_Small" H 1860 6390 50  0000 C CNN
-F 2 "jumper:SOLDER-JUMPER_1-WAY" H 1850 6450 50  0001 C CNN
+F 2 "SolderJumpers-Tim:SJ_1_NO" H 1850 6450 50  0001 C CNN
 F 3 "" H 1850 6450 50  0000 C CNN
 	1    1850 6450
@@
 F 0 "JP1" H 1850 4530 50  0000 C CNN
 F 1 "Jumper_NO_Small" H 1860 4390 50  0000 C CNN
-F 2 "jumper:SOLDER-JUMPER_1-WAY" H 1850 4450 50  0001 C CNN
+F 2 "SolderJumpers-Tim:SJ_1_NO" H 1850 4450 50  0001 C CNN
 F 3 "" H 1850 4450 50  0000 C CNN
 	1    1850 4450
@@
 F 0 "JP2" H 1850 4630 50  0000 C CNN
 F 1 "Jumper_NO_Small" H 1860 4490 50  0000 C CNN
-F 2 "jumper:SOLDER-JUMPER_1-WAY" H 1850 4550 50  0001 C CNN
+F 2 "SolderJumpers-Tim:SJ_1_NO" H 1850 4550 50  0001 C CNN
 F 3 "" H 1850 4550 50  0000 C CNN
 	1    1850 4550
@@
 F 0 "JP3" H 1850 4730 50  0000 C CNN
 F 1 "Jumper_NO_Small" H 1860 4590 50  0000 C CNN
-F 2 "jumper:SOLDER-JUMPER_1-WAY" H 1850 4650 50  0001 C CNN
+F 2 "SolderJumpers-Tim:SJ_1_NO" H 1850 4650 50  0001 C CNN
 F 3 "" H 1850 4650 50  0000 C CNN
 	1    1850 4650
@@
 F 0 "JP8" H 8800 2080 50  0000 C CNN
 F 1 "Jumper_NO_Small" H 8810 1940 50  0000 C CNN
-F 2 "jumper:SOLDER-JUMPER_1-WAY" H 8800 2000 50  0001 C CNN
+F 2 "SolderJumpers-Tim:SJ_1_NO" H 8800 2000 50  0001 C CNN
 F 3 "" H 8800 2000 50  0000 C CNN
 	1    8800 2000
@@
 F 0 "JP7" H 8800 1980 50  0000 C CNN
 F 1 "Jumper_NO_Small" H 8810 1840 50  0000 C CNN
-F 2 "jumper:SOLDER-JUMPER_1-WAY" H 8800 1900 50  0001 C CNN
+F 2 "SolderJumpers-Tim:SJ_1_NO" H 8800 1900 50  0001 C CNN
 F 3 "" H 8800 1900 50  0000 C CNN
 	1    8800 1900
