File: step_down_led_board.kicad_pcb (KiCad board)
At the start: 2 copper layers, 29.2 x 50.8 mm, 34 parts, among them CON1 BARREL_JACK, J1 OSHW Logo, J2 Polarity Mark, M1 BuckModule, M2 BuckModule, P1 CONN_02X20, P2 CONN_01X02, P3 CONN_01X05, P4 CONN_01X02, P5 CONN_01X02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

Commit message: Use my solder jumper part.
Also fix some trace stragglers and silkscreen.
Parts:
- JP1, JP2, JP3, JP4, JP5, JP6, JP7, JP8: footprint jumper:SOLDER-JUMPER_1-WAY -> SolderJumpers-Tim:SJ_1_NO
Routing:
- net (no net): track 2.20 -> 0.00 mm
Other:
- board text removed: "Center +"

Commit message: Add v0.2 text
Other:
- board text added: "v0.2"
Changed lines of the file:
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@@
     (area 140.575 70.229999 175.213334 128.104048)
     (thickness 1.6)
-    (drawings 17)
+    (drawings 18)
     (tracks 216)
     (zones 0)
@@
   (page A4)
   (layers
-    (0 F.Cu signal hide)
-    (31 B.Cu signal hide)
+    (0 F.Cu signal)
+    (31 B.Cu signal)
     (32 B.Adhes user)
     (33 F.Adhes user)
@@
     (descr "Through hole straight pin header, 2x20, 2.54mm pitch, double rows")
     (tags "Through hole pin header THT 2x20 2.54mm double row")
-    (fp_text reference P1 (at -2.54 0 90) (layer F.SilkS)
+    (fp_text reference P1 (at -5.715 0 90) (layer F.SilkS)
       (effects (font (size 1 1) (thickness 0.15)))
     )
@@
     (descr "Through hole straight pin header, 1x06, 2.54mm pitch, single row")
     (tags "Through hole pin header THT 1x06 2.54mm single row")
-    (fp_text reference P9 (at 0 -2.33) (layer F.SilkS)
+    (fp_text reference P9 (at -3.81 0 90) (layer F.SilkS)
       (effects (font (size 1 1) (thickness 0.15)))
     )
@@
     (fp_line (start 1.8 14.5) (end 1.8 -1.8) (layer F.CrtYd) (width 0.05))
     (fp_line (start 1.8 -1.8) (end -1.8 -1.8) (layer F.CrtYd) (width 0.05))
-    (fp_text user %R (at 0 -2.33) (layer F.Fab)
+    (fp_text user %R (at -3.81 0 90) (layer F.Fab)
       (effects (font (size 1 1) (thickness 0.15)))
     )
@@
       (net 18 "Net-(JP8-Pad2)"))
   )
+  (gr_text v0.2 (at 147.32 76.835) (layer F.SilkS)
+    (effects (font (size 1.5 1.5) (thickness 0.3)))
+  )
   (gr_text timhatch.com/projects/pi-fets (at 145.415 87.63 270) (layer F.SilkS)
