File: buck.sch (KiCad schematic (older format))
At the start: 12 parts, among them U201 MP2315

Commit message: Massive changes, including makefile
Parts:
- C202, C203: footprint Capacitors_SMD_Round:C_0603 -> Capacitors_SMD:C_0603
Changed lines of the file:
@@
 $Descr A4 11693 8268
 encoding utf-8
-Sheet 3 3
+Sheet 2 3
 Title ""
 Date ""
@@
 AR Path="/5A895547/5A8957D8" Ref="U201"  Part="1"
 AR Path="/5A89570E/5A8957D8" Ref="U301"  Part="1"
-F 0 "U301" H 5400 3700 60  0000 C CNN
+F 0 "U201" H 5400 3700 60  0000 C CNN
 F 1 "MP2315" H 5650 3350 60  0000 C CNN
 F 2 "TO_SOT_Packages_SMD:SOT-23-8" H 5650 3200 60  0001 C CNN
@@
 AR Path="/5A895547/5A895834" Ref="C201"  Part="1"
 AR Path="/5A89570E/5A895834" Ref="C301"  Part="1"
-F 0 "C301" H 4475 3650 50  0000 L CNN
+F 0 "C201" H 4475 3650 50  0000 L CNN
 F 1 "22u" H 4475 3450 50  0000 L CNN
 F 2 "Capacitors_SMD_Round:C_1206" H 4488 3400 50  0001 C CNN
@@
 AR Path="/5A895547/5A89588A" Ref="#PWR201"  Part="1"
 AR Path="/5A89570E/5A89588A" Ref="#PWR301"  Part="1"
-F 0 "#PWR301" H 4450 3750 50  0001 C CNN
+F 0 "#PWR201" H 4450 3750 50  0001 C CNN
 F 1 "GND" H 4450 3850 50  0000 C CNN
 F 2 "" H 4450 4000 50  0001 C CNN
@@
 AR Path="/5A895547/5A8958A2" Ref="R201"  Part="1"
 AR Path="/5A89570E/5A8958A2" Ref="R301"  Part="1"
-F 0 "R301" V 5030 3200 50  0000 C CNN
+F 0 "R201" V 5030 3200 50  0000 C CNN
 F 1 "100k" V 4950 3200 50  0000 C CNN
 F 2 "Resistors_SMD:R_0603" V 4880 3200 50  0001 C CNN
@@
 AR Path="/5A895547/5A8958F7" Ref="C202"  Part="1"
 AR Path="/5A89570E/5A8958F7" Ref="C302"  Part="1"
-F 0 "C302" H 4775 3650 50  0000 L CNN
+F 0 "C202" H 4775 3650 50  0000 L CNN
 F 1 "0.1u" H 4775 3450 50  0000 L CNN
-F 2 "Capacitors_SMD_Round:C_0603" H 4788 3400 50  0001 C CNN
+F 2 "Capacitors_SMD:C_0603" H 4788 3400 50  0001 C CNN
 F 3 "" H 4750 3550 50  0001 C CNN
 	1    4750 3550
@@
 AR Path="/5A895547/5A895936" Ref="R202"  Part="1"
 AR Path="/5A89570E/5A895936" Ref="R302"  Part="1"
-F 0 "R302" V 5130 3750 50  0000 C CNN
+F 0 "R202" V 5130 3750 50  0000 C CNN
 F 1 "75k" V 5050 3750 50  0000 C CNN
 F 2 "Resistors_SMD:R_0603" V 4980 3750 50  0001 C CNN
@@
 AR Path="/5A895547/5A895972" Ref="#PWR203"  Part="1"
 AR Path="/5A89570E/5A895972" Ref="#PWR303"  Part="1"
-F 0 "#PWR303" H 5050 3750 50  0001 C CNN
+F 0 "#PWR203" H 5050 3750 50  0001 C CNN
 F 1 "GND" H 5050 3850 50  0000 C CNN
 F 2 "" H 5050 4000 50  0001 C CNN
@@
 AR Path="/5A895547/5A8959AC" Ref="#PWR202"  Part="1"
 AR Path="/5A89570E/5A8959AC" Ref="#PWR302"  Part="1"
-F 0 "#PWR302" H 4750 3750 50  0001 C CNN
+F 0 "#PWR202" H 4750 3750 50  0001 C CNN
 F 1 "GND" H 4750 3850 50  0000 C CNN
 F 2 "" H 4750 4000 50  0001 C CNN
@@
 AR Path="/5A895547/5A895C8C" Ref="R203"  Part="1"
 AR Path="/5A89570E/5A895C8C" Ref="R303"  Part="1"
-F 0 "R303" V 6480 2900 50  0000 C CNN
+F 0 "R203" V 6480 2900 50  0000 C CNN
 F 1 "20R" V 6400 2900 50  0000 C CNN
 F 2 "Resistors_SMD:R_0603" V 6330 2900 50  0001 C CNN
@@
 AR Path="/5A895547/5A895CB5" Ref="C203"  Part="1"
 AR Path="/5A89570E/5A895CB5" Ref="C303"  Part="1"
-F 0 "C303" H 6725 3150 50  0000 L CNN
+F 0 "C203" H 6725 3150 50  0000 L CNN
 F 1 "0.1u" H 6725 2950 50  0000 L CNN
-F 2 "Capacitors_SMD_Round:C_0603" H 6738 2900 50  0001 C CNN
+F 2 "Capacitors_SMD:C_0603" H 6738 2900 50  0001 C CNN
 F 3 "" H 6700 3050 50  0001 C CNN
 	1    6700 3050
@@
 AR Path="/5A895547/5A895EA3" Ref="R204"  Part="1"
 AR Path="/5A89570E/5A895EA3" Ref="R304"  Part="1"
-F 0 "R304" V 6530 3500 50  0000 C CNN
+F 0 "R204" V 6530 3500 50  0000 C CNN
 F 1 "R" V 6450 3500 50  0000 C CNN
 F 2 "Resistors_SMD:R_0603" V 6380 3500 50  0001 C CNN
@@
 AR Path="/5A895547/5A895F12" Ref="R206"  Part="1"
 AR Path="/5A89570E/5A895F12" Ref="R306"  Part="1"
-F 0 "R306" V 7530 3700 50  0000 C CNN
+F 0 "R206" V 7530 3700 50  0000 C CNN
 F 1 "R" V 7450 3700 50  0000 C CNN
 F 2 "Resistors_SMD:R_0603" V 7380 3700 50  0001 C CNN
@@
 AR Path="/5A895547/5A895F4F" Ref="L201"  Part="1"
 AR Path="/5A89570E/5A895F4F" Ref="L301"  Part="1"
-F 0 "L301" V 7050 3200 50  0000 C CNN
+F 0 "L201" V 7050 3200 50  0000 C CNN
 F 1 "L" V 7175 3200 50  0000 C CNN
 F 2 "Inductors_SMD:L_Taiyo-Yuden_MD-5050" H 7100 3200 50  0001 C CNN
@@
 AR Path="/5A895547/5A895FC6" Ref="R205"  Part="1"
 AR Path="/5A89570E/5A895FC6" Ref="R305"  Part="1"
-F 0 "R305" V 7530 3350 50  0000 C CNN
+F 0 "R205" V 7530 3350 50  0000 C CNN
 F 1 "R" V 7450 3350 50  0000 C CNN
 F 2 "Resistors_SMD:R_0603" V 7380 3350 50  0001 C CNN
@@
 AR Path="/5A895547/5A89605E" Ref="#PWR205"  Part="1"
 AR Path="/5A89570E/5A89605E" Ref="#PWR305"  Part="1"
-F 0 "#PWR305" H 7450 3650 50  0001 C CNN
+F 0 "#PWR205" H 7450 3650 50  0001 C CNN
 F 1 "GND" H 7450 3750 50  0000 C CNN
 F 2 "" H 7450 3900 50  0001 C CNN
@@
 AR Path="/5A895547/5A89614A" Ref="#PWR206"  Part="1"
 AR Path="/5A89570E/5A89614A" Ref="#PWR306"  Part="1"
-F 0 "#PWR306" H 7850 3350 50  0001 C CNN
+F 0 "#PWR206" H 7850 3350 50  0001 C CNN
 F 1 "GND" H 7850 3450 50  0000 C CNN
 F 2 "" H 7850 3600 50  0001 C CNN
@@
 AR Path="/5A895547/5A8994BC" Ref="#PWR204"  Part="1"
 AR Path="/5A89570E/5A8994BC" Ref="#PWR304"  Part="1"
-F 0 "#PWR304" H 5650 3750 50  0001 C CNN
+F 0 "#PWR204" H 5650 3750 50  0001 C CNN
 F 1 "GND" H 5650 3850 50  0000 C CNN
 F 2 "" H 5650 4000 50  0001 C CNN
@@
 AR Path="/5A89570E/5A89E5E0" Ref="C304"  Part="1"
 AR Path="/5A895547/5A89E5E0" Ref="C204"  Part="1"
-F 0 "C304" H 7950 3450 60  0000 C CNN
+F 0 "C204" H 7950 3450 60  0000 C CNN
 F 1 "44u" H 8000 3250 60  0000 C CNN
 F 2 "Capacitors_SMD_Round:C_1206_NetTie" H 7850 3350 60  0001 C CNN
